File: ice4pi.kicad_pcb (KiCad board)
At the start: 4 copper layers, 85 x 54 mm, 43 parts, among them J1 Conn_02x20_Odd_Even, J2 Conn_01x01_Shielded, J4 Conn_02x20_Odd_Even, J5 Conn_01x01_Shielded, J6 Conn_01x01_Shielded, M0 MountingHole_2.7mm_Pad, M1 MountingHole_2.7mm_Pad, M2 MountingHole_2.7mm_Pad, Q1 Q_NPN_BEC_BRT, U1 74LVC1G125, U10 PCA9306, U2 74LVC1G125, U3 SN74LV1T34DBVRG4, U4 SN74LV1T34DBVRG4, U5 LD1117S33TR_SOT223, U6 LEA-M8T, U7 SN74LV1T34DBVRG4, U8 SN74LV1T34DBVRG4, U9 SN74LV1T34DBVRG4

Commit message: Release gnssclock496boards-1.0
Parts:
- removed the svg2mod at (97.4, 53.6)
- added svg2mod: G***, ice4pi:lsi-logo-24mm, F.Cu at (59.1, 100.0)
- R1, R2: footprint Resistor_SMD:R_0402_1005Metric -> Resistor_SMD:R_0805_2012Metric
- R6: footprint Resistor_SMD:R_0603_1608Metric -> Resistor_SMD:R_0402_1005Metric
Connections:
- U6 pad 1: (no net) -> unconnected-(U6-Pad1)
- U6 pad 2: (no net) -> unconnected-(U6-Pad2)
- U6 pad 20: (no net) -> unconnected-(U6-Pad20)
- U6 pad 21: (no net) -> unconnected-(U6-Pad21)
- U6 pad 22: (no net) -> unconnected-(U6-Pad22)
- U6 pad 23: (no net) -> unconnected-(U6-Pad23)
- U6 pad 25: (no net) -> unconnected-(U6-Pad25)
- U6 pad 26: (no net) -> unconnected-(U6-Pad26)
- U6 pad 27: (no net) -> unconnected-(U6-Pad27)
- U6 pad 5: (no net) -> unconnected-(U6-Pad5)
- U6 pad 8: (no net) -> unconnected-(U6-Pad8)
- U6 pad 9: (no net) -> unconnected-(U6-Pad9)
Routing:
- net Net-(R1-Pad2): track 34.9 -> 34.1 mm
Other:
- board text added: "10MHz OUT"
- board text added: "1PPS OUT"
- board text added: "CR2450 battery"
- board text added: "RF IN"
- board text added: "gnssclock496boards-1.0"
- board text removed: "1"
- board text removed: "P/N:"
- board text removed: "REV:"
- board text removed: "gpsclock4ultra96-1"

Commit message: Release gnssclock496boards-2.0
Parts:
- moved D1 3.90 mm to (78.0, 58.4)
- moved R1 3.80 mm to (78.0, 60.2)
- moved J5 3.38 mm to (78.0, 53.6)
- moved BT1 2.75 mm to (68.0, 76.7)
- moved D2 2.60 mm to (58.0, 58.5)
- moved R2 2.60 mm to (58.0, 60.2)
- moved J2 2.50 mm to (116.0, 53.6)
- moved J6 2.12 mm to (58.0, 53.6)
- moved L1 1.58 mm to (119.5, 60.1), turned to -90 degrees
Routing:
- net Net-(R1-Pad2): track 34.1 -> 38.7 mm, vias 0 -> 2
- net Net-(BT1-Pad1): track 52.6 -> 55.4 mm
- net Net-(R2-Pad2): track 55.8 -> 57.9 mm
- net Net-(L1-Pad2): track 3.61 -> 1.55 mm
- net Net-(C4-Pad2): track 11.0 -> 12.5 mm
Other:
- board text added: "gnssclock496boards-2.0"
- board text removed: "gnssclock496boards-1.0"

Commit message: Release gnssclock496boards-2.1
Parts:
- added 1: Fiducial_1mm_Mask3mm, Fiducial:Fiducial_1mm_Mask3mm, F.Cu at (53.5, 92.5)
- added 2: Fiducial_1mm_Mask3mm, Fiducial:Fiducial_1mm_Mask3mm, F.Cu at (130.5, 52.0)
Other:
- board text added: "gnssclock496boards-2.1"
- board text removed: "gnssclock496boards-2.0"
Changed lines of the file:
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@@
   (paper "A4")
   (title_block
-    (title "gnssclock496boards-2.0")
+    (title "gnssclock496boards-2.1")
     (company "Lightside Instruments AS")
   )
@@
       ) (layer "F.Mask") (width 0) (fill solid))
   )
+  (footprint "Fiducial:Fiducial_1mm_Mask3mm" (layer "F.Cu")
+    (at 53.5 92.5)
+    (descr "Circular Fiducial, 1mm bare copper, 3mm soldermask opening (recommended)")
+    (tags "fiducial")
+    (attr smd)
+    (fp_text reference "1" (at -2.5 0) (layer "F.SilkS")
+      (effects (font (size 1 1) (thickness 0.15)))
+    )
+    (fp_text value "Fiducial_1mm_Mask3mm" (at 0 2.286) (layer "F.Fab")
+      (effects (font (size 1 1) (thickness 0.15)))
+    )
+    (fp_text user "${REFERENCE}" (at 0 0) (layer "F.Fab")
+      (effects (font (size 0.4 0.4) (thickness 0.06)))
+    )
+    (fp_circle (center 0 0) (end 1.75 0) (layer "F.CrtYd") (width 0.05) (fill none))
+    (fp_circle (center 0 0) (end 1.5 0) (layer "F.Fab") (width 0.1) (fill none))
+    (pad "" smd circle (at 0 0) (size 1 1) (layers "F.Cu" "F.Mask")
+      (solder_mask_margin 1) (clearance 1))
+  )
+  (footprint "Fiducial:Fiducial_1mm_Mask3mm" (layer "F.Cu")
+    (at 130.5 52)
+    (descr "Circular Fiducial, 1mm bare copper, 3mm soldermask opening (recommended)")
+    (tags "fiducial")
+    (attr smd board_only exclude_from_pos_files exclude_from_bom)
+    (fp_text reference "2" (at 2.5 0) (layer "F.SilkS")
+      (effects (font (size 1 1) (thickness 0.15)))
+    )
+    (fp_text value "Fiducial_1mm_Mask3mm" (at 0 1.5) (layer "F.Fab")
+      (effects (font (size 1 1) (thickness 0.15)))
+    )
+    (fp_text user "${REFERENCE}" (at 0 0) (layer "F.Fab")
+      (effects (font (size 0.4 0.4) (thickness 0.06)))
+    )
+    (fp_circle (center 0 0) (end 1.75 0) (layer "F.CrtYd") (width 0.05) (fill none))
+    (fp_circle (center 0 0) (end 1.5 0) (layer "F.Fab") (width 0.1) (fill none))
+    (pad "" smd circle (at 0 0) (size 1 1) (layers "F.Cu" "F.Mask")
+      (solder_mask_margin 1) (clearance 1))
+  )
   (footprint "ice4pi:Pin_Header_SMD_2x20_Pitch2mm" (layer "B.Cu")
     (at 124.5 97.5 90)
@@
     )
   )
+  (gr_line (start 92 77.5) (end 92 73.5) (layer "B.SilkS") (width 0.12))
+  (gr_line (start 90 75.5) (end 94 75.5) (layer "B.SilkS") (width 0.12))
+  (gr_line (start 92 77.5) (end 92 73.5) (layer "F.SilkS") (width 0.12))
+  (gr_line (start 90 75.5) (end 94 75.5) (layer "F.SilkS") (width 0.12))
   (gr_line (start 49.5 48.5) (end 134.5 48.5) (layer "Edge.Cuts") (width 0.05))
   (gr_line (start 134.5 48.5) (end 134.5 102.5) (layer "Edge.Cuts") (width 0.05))
   (gr_line (start 49.5 102.5) (end 134.5 102.5) (layer "Edge.Cuts") (width 0.05))
   (gr_line (start 49.5 48.5) (end 49.5 102.5) (layer "Edge.Cuts") (width 0.05))
-  (gr_text "gnssclock496boards-2.0" (at 68.5 99) (layer "F.SilkS")
+  (gr_text "gnssclock496boards-2.1" (at 68.5 99) (layer "F.SilkS")
     (effects (font (size 1 1) (thickness 0.25)))
   )
