File: ice4pi.kicad_sch (KiCad schematic)
At the start: 38 parts, among them J1 Conn_02x20_Odd_Even, J2 Conn_01x01_Shielded, J4 Conn_02x20_Odd_Even, J5 Conn_01x01_Shielded, J6 Conn_01x01_Shielded, Q1 Q_NPN_BEC_BRT, U1 74LVC1G125, U10 PCA9306, U2 74LVC1G125, U3 SN74LV1T34DBVRG4, U4 SN74LV1T34DBVRG4, U5 LD1117S33TR_SOT223, U6 LEA-M8T, U7 SN74LV1T34DBVRG4, U8 SN74LV1T34DBVRG4, U9 SN74LV1T34DBVRG4

Commit message: Release gnssclock496boards-1.0
Parts:
- R1, R2: footprint Resistor_SMD:R_0402_1005Metric -> Resistor_SMD:R_0805_2012Metric
- R6: footprint Resistor_SMD:R_0603_1608Metric -> Resistor_SMD:R_0402_1005Metric
Connections:
- net +3.3V is gone; now on net +3V3: R10.2, R11.2, R9.2
Other:
- title: gpsclock4ultra96 ver. 1 -> gnssclock496boards-1.0
Changed lines of the file:
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@@
   (paper "A3")
   (title_block
-    (title "gpsclock4ultra96 ver. 1")
-    (date "2021-09-08")
-    (rev "1")
+    (title "gnssclock496boards-1.0")
     (company "Lightside Instruments AS")
   )
@@
   (junction (at 195.58 67.31) (diameter 0) (color 0 0 0 0)
   )
+  (junction (at 87.63 186.69) (diameter 0) (color 0 0 0 0)
+  )
+  (junction (at 227.33 130.81) (diameter 0) (color 0 0 0 0)
+  )
+  (junction (at 60.96 194.31) (diameter 0) (color 0 0 0 0)
+  )
+  (junction (at 317.5 198.12) (diameter 0) (color 0 0 0 0)
+  )
+  (junction (at 212.09 74.93) (diameter 0) (color 0 0 0 0)
+  )
+  (junction (at 54.61 209.55) (diameter 0) (color 0 0 0 0)
+  )
+  (junction (at 309.88 190.5) (diameter 0) (color 0 0 0 0)
+  )
+  (junction (at 76.2 194.31) (diameter 0) (color 0 0 0 0)
+  )
+  (junction (at 325.12 190.5) (diameter 0) (color 0 0 0 0)
+  )
+  (junction (at 92.71 146.05) (diameter 0) (color 0 0 0 0)
+  )
+  (junction (at 322.58 96.52) (diameter 0) (color 0 0 0 0)
+  )
+  (junction (at 49.53 143.51) (diameter 0) (color 0 0 0 0)
+  )
+  (junction (at 87.63 207.01) (diameter 0) (color 0 0 0 0)
+  )
+  (junction (at 93.98 209.55) (diameter 0) (color 0 0 0 0)
+  )
+  (junction (at 242.57 62.23) (diameter 0) (color 0 0 0 0)
+  )
+  (junction (at 60.96 207.01) (diameter 0) (color 0 0 0 0)
+  )
+  (junction (at 71.12 194.31) (diameter 0) (color 0 0 0 0)
+  )
   (junction (at 76.2 186.69) (diameter 0) (color 0 0 0 0)
-  )
-  (junction (at 87.63 186.69) (diameter 0) (color 0 0 0 0)
-  )
-  (junction (at 227.33 130.81) (diameter 0) (color 0 0 0 0)
-  )
-  (junction (at 60.96 194.31) (diameter 0) (color 0 0 0 0)
-  )
-  (junction (at 317.5 198.12) (diameter 0) (color 0 0 0 0)
-  )
-  (junction (at 212.09 74.93) (diameter 0) (color 0 0 0 0)
-  )
-  (junction (at 54.61 209.55) (diameter 0) (color 0 0 0 0)
-  )
-  (junction (at 309.88 190.5) (diameter 0) (color 0 0 0 0)
-  )
-  (junction (at 76.2 194.31) (diameter 0) (color 0 0 0 0)
-  )
-  (junction (at 325.12 190.5) (diameter 0) (color 0 0 0 0)
-  )
-  (junction (at 92.71 146.05) (diameter 0) (color 0 0 0 0)
-  )
-  (junction (at 322.58 96.52) (diameter 0) (color 0 0 0 0)
-  )
-  (junction (at 49.53 143.51) (diameter 0) (color 0 0 0 0)
-  )
-  (junction (at 87.63 207.01) (diameter 0) (color 0 0 0 0)
-  )
-  (junction (at 93.98 209.55) (diameter 0) (color 0 0 0 0)
-  )
-  (junction (at 242.57 62.23) (diameter 0) (color 0 0 0 0)
-  )
-  (junction (at 60.96 207.01) (diameter 0) (color 0 0 0 0)
-  )
-  (junction (at 71.12 194.31) (diameter 0) (color 0 0 0 0)
   )
   (junction (at 49.53 110.49) (diameter 0) (color 0 0 0 0)
@@
     (pin "1")
   )
-  (symbol (lib_id "power:+3.3V") (at 76.2 186.69 0) (mirror y) (unit 1)
-    (in_bom yes) (on_board yes)
-    (property "Reference" "#PWR0188" (id 0) (at 76.2 190.5 0)
-      (effects (font (size 1.27 1.27)) hide)
-    )
-    (property "Value" "+3.3V" (id 1) (at 75.819 182.2958 90))
-    (property "Footprint" "" (id 2) (at 76.2 186.69 0)
-      (effects (font (size 1.27 1.27)) hide)
-    )
-    (property "Datasheet" "" (id 3) (at 76.2 186.69 0)
-      (effects (font (size 1.27 1.27)) hide)
-    )
-    (pin "1")
-  )
   (symbol (lib_id "Device:R") (at 76.2 190.5 0) (mirror x) (unit 1)
     (in_bom yes) (on_board yes)
@@
     (property "Reference" "R1" (id 0) (at 55.88 138.2522 90))
     (property "Value" "51" (id 1) (at 55.88 140.5636 90))
-    (property "Footprint" "Resistor_SMD:R_0402_1005Metric" (id 2) (at 55.88 141.732 90)
+    (property "Footprint" "Resistor_SMD:R_0805_2012Metric" (id 2) (at 55.88 141.732 90)
       (effects (font (size 1.27 1.27)) hide)
     )
@@
     (property "Reference" "R2" (id 0) (at 55.88 105.2322 90))
     (property "Value" "51" (id 1) (at 55.88 107.5436 90))
-    (property "Footprint" "Resistor_SMD:R_0402_1005Metric" (id 2) (at 55.88 108.712 90)
+    (property "Footprint" "Resistor_SMD:R_0805_2012Metric" (id 2) (at 55.88 108.712 90)
       (effects (font (size 1.27 1.27)) hide)
     )
@@
     (in_bom yes) (on_board yes)
     (property "Reference" "U1" (id 0) (at 69.85 135.89 0))
-    (property "Value" "74LVC1G125" (id 1) (at 62.23 130.81 0))
+    (property "Value" "74LVC1G125" (id 1) (at 64.77 153.67 0))
     (property "Footprint" "Package_SO:TSOP-5_1.65x3.05mm_P0.95mm" (id 2) (at 72.39 143.51 0)
       (effects (font (size 1.27 1.27)) hide)
@@
     (in_bom yes) (on_board yes)
     (property "Reference" "U2" (id 0) (at 69.85 102.87 0))
-    (property "Value" "74LVC1G125" (id 1) (at 62.23 99.06 0))
+    (property "Value" "74LVC1G125" (id 1) (at 64.77 120.65 0))
     (property "Footprint" "Package_SO:TSOP-5_1.65x3.05mm_P0.95mm" (id 2) (at 72.39 110.49 0)
       (effects (font (size 1.27 1.27)) hide)
@@
   (symbol (lib_id "ice4pi:SN74LV1T34DBVRG4") (at 109.22 146.05 0) (unit 1)
     (in_bom yes) (on_board yes)
-    (property "Reference" "U3" (id 0) (at 120.4214 144.8816 0)
-      (effects (font (size 1.27 1.27)) (justify left))
-    )
-    (property "Value" "SN74LV1T34DBVRG4" (id 1) (at 120.4214 147.193 0)
+    (property "Reference" "U3" (id 0) (at 114.3 139.7 0)
+      (effects (font (size 1.27 1.27)) (justify left))
+    )
+    (property "Value" "SN74LV1T34DBVRG4" (id 1) (at 113.03 152.4 0)
       (effects (font (size 1.27 1.27)) (justify left))
     )
@@
   (symbol (lib_id "ice4pi:SN74LV1T34DBVRG4") (at 107.95 113.03 0) (unit 1)
     (in_bom yes) (on_board yes)
-    (property "Reference" "U8" (id 0) (at 119.1514 111.8616 0)
-      (effects (font (size 1.27 1.27)) (justify left))
-    )
-    (property "Value" "SN74LV1T34DBVRG4" (id 1) (at 119.1514 114.173 0)
+    (property "Reference" "U8" (id 0) (at 113.03 106.68 0)
+      (effects (font (size 1.27 1.27)) (justify left))
+    )
+    (property "Value" "SN74LV1T34DBVRG4" (id 1) (at 110.49 119.38 0)
       (effects (font (size 1.27 1.27)) (justify left))
     )
@@
   (symbol (lib_id "ice4pi:SN74LV1T34DBVRG4") (at 107.95 57.15 0) (unit 1)
     (in_bom yes) (on_board yes)
-    (property "Reference" "U4" (id 0) (at 119.1514 55.9816 0)
-      (effects (font (size 1.27 1.27)) (justify left))
-    )
-    (property "Value" "SN74LV1T34DBVRG4" (id 1) (at 119.1514 58.293 0)
+    (property "Reference" "U4" (id 0) (at 113.03 50.8 0)
+      (effects (font (size 1.27 1.27)) (justify left))
+    )
+    (property "Value" "SN74LV1T34DBVRG4" (id 1) (at 110.49 63.5 0)
       (effects (font (size 1.27 1.27)) (justify left))
     )
@@
   (symbol (lib_id "ice4pi:SN74LV1T34DBVRG4") (at 107.95 85.09 0) (mirror y) (unit 1)
     (in_bom yes) (on_board yes)
-    (property "Reference" "U7" (id 0) (at 96.7486 83.9216 0)
-      (effects (font (size 1.27 1.27)) (justify left))
-    )
-    (property "Value" "SN74LV1T34DBVRG4" (id 1) (at 96.7486 86.233 0)
+    (property "Reference" "U7" (id 0) (at 114.3 78.74 0)
+      (effects (font (size 1.27 1.27)) (justify left))
+    )
+    (property "Value" "SN74LV1T34DBVRG4" (id 1) (at 129.54 91.44 0)
       (effects (font (size 1.27 1.27)) (justify left))
     )
@@
       (effects (font (size 1.27 1.27)) (justify left))
     )
-    (property "Footprint" "Resistor_SMD:R_0603_1608Metric" (id 2) (at 235.712 114.3 90)
+    (property "Footprint" "Resistor_SMD:R_0402_1005Metric" (id 2) (at 235.712 114.3 90)
       (effects (font (size 1.27 1.27)) hide)
     )
@@
   (symbol (lib_id "ice4pi:SN74LV1T34DBVRG4") (at 184.15 143.51 0) (mirror y) (unit 1)
     (in_bom yes) (on_board yes)
-    (property "Reference" "U9" (id 0) (at 195.3514 142.3416 0)
+    (property "Reference" "U9" (id 0) (at 189.23 137.16 0)
       (effects (font (size 1.27 1.27)) (justify right))
     )
-    (property "Value" "SN74LV1T34DBVRG4" (id 1) (at 195.3514 144.653 0)
+    (property "Value" "SN74LV1T34DBVRG4" (id 1) (at 185.42 149.86 0)
       (effects (font (size 1.27 1.27)) (justify right))
     )
@@
     (pin "2")
   )
+  (symbol (lib_id "power:+3V3") (at 76.2 186.69 0) (unit 1)
+    (in_bom yes) (on_board yes)
+    (property "Reference" "#PWR0135" (id 0) (at 76.2 190.5 0)
+      (effects (font (size 1.27 1.27)) hide)
+    )
+    (property "Value" "+3V3" (id 1) (at 76.581 182.2958 0))
+    (property "Footprint" "" (id 2) (at 76.2 186.69 0)
+      (effects (font (size 1.27 1.27)) hide)
+    )
+    (property "Datasheet" "" (id 3) (at 76.2 186.69 0)
+      (effects (font (size 1.27 1.27)) hide)
+    )
+    (pin "1")
+  )
   (sheet_instances
     (path "/" (page "1"))
@@
       (reference "#PWR0134") (unit 1) (value "GND") (footprint "")
     )
+    (path "/bc1e4e93-ff30-4601-ac32-2b96f6c04cfc"
+      (reference "#PWR0135") (unit 1) (value "+3V3") (footprint "")
+    )
     (path "/00000000-0000-0000-0000-000060e0090e"
       (reference "#PWR0138") (unit 1) (value "GND") (footprint "")
@@
       (reference "#PWR0187") (unit 1) (value "+1V8") (footprint "")
     )
-    (path "/00000000-0000-0000-0000-0000611cf1e2"
-      (reference "#PWR0188") (unit 1) (value "+3.3V") (footprint "")
-    )
     (path "/00000000-0000-0000-0000-000061367e39"
       (reference "BT1") (unit 1) (value "Battery_Cell") (footprint "ice4pi:BatteryHolder_Keystone_2450")
@@
     )
     (path "/00000000-0000-0000-0000-0000612e33b5"
-      (reference "R1") (unit 1) (value "51") (footprint "Resistor_SMD:R_0402_1005Metric")
+      (reference "R1") (unit 1) (value "51") (footprint "Resistor_SMD:R_0805_2012Metric")
     )
     (path "/00000000-0000-0000-0000-0000612e4bab"
-      (reference "R2") (unit 1) (value "51") (footprint "Resistor_SMD:R_0402_1005Metric")
+      (reference "R2") (unit 1) (value "51") (footprint "Resistor_SMD:R_0805_2012Metric")
     )
     (path "/00000000-0000-0000-0000-00006138c87e"
@@
     )
     (path "/00000000-0000-0000-0000-000061357a03"
-      (reference "R6") (unit 1) (value "1K") (footprint "Resistor_SMD:R_0603_1608Metric")
+      (reference "R6") (unit 1) (value "1K") (footprint "Resistor_SMD:R_0402_1005Metric")
     )
     (path "/00000000-0000-0000-0000-00006134158a"

Commit message: Release gnssclock496boards-2.0
Other:
- title: gnssclock496boards-1.0 -> gnssclock496boards-2.0
Changed lines of the file:
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@@
   (paper "A3")
   (title_block
-    (title "gnssclock496boards-1.0")
+    (title "gnssclock496boards-2.0")
     (company "Lightside Instruments AS")
   )

Commit message: Release gnssclock496boards-2.1
Other:
- title: gnssclock496boards-2.0 -> gnssclock496boards-2.1
Changed lines of the file:
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@@
   (paper "A3")
   (title_block
-    (title "gnssclock496boards-2.0")
+    (title "gnssclock496boards-2.1")
     (company "Lightside Instruments AS")
   )
